Commit message: fix camera orientation

File: install/gazebo_ackermann_steering_vehicle/share/gazebo_ackermann_steering_vehicle/model/vehicle.xacro (robot description, xacro)
@@ -218,27 +218,4 @@
     </inertial>
   </link>
-  <!-- Camera Stick Link -->
-  <link name="camera_stick_link">
-    <collision>
-      <origin xyz="0 0 0" rpy="0 0 0"/>
-      <geometry>
-        <box size="${camera_stick_size} ${camera_stick_size} ${camera_height}"/>
-      </geometry>
-    </collision>
-    <visual>
-      <origin xyz="0 0 0" rpy="0 0 0"/>
-      <geometry>
-        <box size="${camera_stick_size} ${camera_stick_size} ${camera_height}"/>
-      </geometry>
-      <material name="camera_stick_material">
-        <color rgba="0.25 0.25 0.25 1.0"/>
-      </material>
-    </visual>
-    <inertial>
-      <mass value="1e-5" />
-      <origin xyz="0 0 0" rpy="0 0 0"/>
-      <inertia ixx="1e-6" ixy="0" ixz="0" iyy="1e-6" iyz="0" izz="1e-6" />
-    </inertial>
-  </link>
   <!-- Camera Link -->
   <link name="camera_link">
@@ -319,17 +296,9 @@
     <dynamics damping="0.1" friction="0.1"/>
   </joint>
-  <!-- Camera Stick Joint -->
-  <joint name="camera_stick_joint" type="fixed">
-    <axis xyz="0 1 0" />
-    <origin xyz="${body_length/2 - camera_stick_size/2} ${camera_box_size/2 + camera_stick_size/2} ${camera_height/2}" rpy="0.0 0.0 0.0"/>
-    <parent link="body_link"/>
-    <child link="camera_stick_link"/>
-  </joint>
   <!-- Camera Joint -->
   <joint name="camera_joint" type="fixed">
-    <axis xyz="0 1 0" />
-    <origin xyz="0.0 ${-camera_box_size/2 - camera_stick_size/2} ${camera_height/2}" rpy="0 ${camera_pitch} 0"/>
-    <origin xyz="0.0 0.0 0.0" rpy="0 ${camera_pitch} 0"/>
-    <parent link="camera_stick_link"/>
+    <axis xyz="0 0 0" />
+    <origin xyz="${body_length/2} 0.0 ${camera_height/2}" rpy="0 0 0"/>
+    <parent link="body_link"/>
     <child link="camera_link"/>
   </joint>

Commit message: change ugv size

File: install/gazebo_ackermann_steering_vehicle/share/gazebo_ackermann_steering_vehicle/model/vehicle.xacro (robot description, xacro)
@@ -299,5 +299,5 @@
   <joint name="camera_joint" type="fixed">
     <axis xyz="0 0 0" />
-    <origin xyz="${body_length/2} 0.0 ${camera_height/2}" rpy="0 0 0"/>
+    <origin xyz="${body_length/2} 0.0 ${camera_box_size}" rpy="0 0 0"/>
     <parent link="body_link"/>
     <child link="camera_link"/>
@@ -413,5 +413,5 @@
         <frameName>camera_link</frameName>
         <min_depth>0.1</min_depth>
-        <max_depth>100.0</max_depth>
+        <max_depth>5.0</max_depth>
         <!--alwaysOn>true</alwaysOn>
         <updateRate>10.0</updateRate>
